File: pcb/uvm.sch (KiCad schematic (older format))
At the start: 176 parts, among them J1 Barrel_Jack, J2 ICSP, J3 FDTI Serial, U1 ATmega328P-PU, U10 74HC595, U11 74HC595, U12 74HC595, U13 74HC595, U14 74HC595, U15 74HC595, U16 74HC595, U17 74HC595, U18 74HC595, U19 74HC595, U2 23LCV512, U3 L7805, U4 74HC595, U5 74HC595, U6 74HC595, U7 74HC595, U8 74HC595, U9 74HC595, Y1 16MHz

Commit message: Completed Schematic and assigned footprints.
Started PCB layout.
Parts:
- removed D106, D107, D108, D122, D123, D124: LED, symbol Device:LED_Small
- removed RN15: 330, Resistor_THT:R_Array_SIP9, symbol Device:R_Network08
- added R3: 10K, Resistor_THT:R_Axial_DIN0207_L6.3mm_D2.5mm_P10.16mm_Horizontal, symbol Device:R
- added R4, R5: 10K, Resistor_THT:R_Axial_DIN0207_L6.3mm_D2.5mm_P10.16mm_Horizontal, symbol Device:R_Small
- added SW21: RESET, Button_Switch_THT:SW_PUSH_6mm_H5mm, symbol Switch:SW_Push
- added SW22: REG Select, uvm:TOGGLE_SPDT_ON_ON_2MS, symbol Switch:SW_SPDT
- BT1: footprint (none) -> Battery:BatteryHolder_Keystone_105_1x2430
- C1, C4, C5, C6: footprint (none) -> Capacitor_THT:C_Disc_D6.0mm_W2.5mm_P5.00mm
- C2: footprint (none) -> Capacitor_THT:CP_Radial_D8.0mm_P3.80mm
- C3: footprint (none) -> Capacitor_THT:C_Disc_D4.7mm_W2.5mm_P5.00mm
- D1, D10, D100, D101, D102, D103, D104, D105, D109, D11, D110, D111, D112, D113, D114, D115, D116, D117, D118, D119, D12, D120, D121, D125, D126, D127, D128, D13, D14, D15, D16, D17, D18, D19, D2, D20, D21, D22, D23, D24, D25, D26, D27, D28, D29, D3, D30, D31, D32, D33, D34, D35, D36, D37, D38, D39, D4, D40, D41, D42, D43, D44, D45, D46, D47, D48, D49, D5, D50, D51, D52, D53, D54, D55, D56, D57, D58, D59, D6, D60, D61, D62, D63, D64, D65, D66, D67, D68, D69, D7, D70, D71, D72, D73, D74, D75, D76, D77, D78, D79, D8, D80, D81, D82, D83, D84, D85, D86, D87, D88, D89, D9, D90, D91, D92, D93, D94, D95, D96, D97, D98, D99: footprint (none) -> LED_THT:LED_D5.0mm
- J1: footprint (none) -> Connector_BarrelJack:BarrelJack_Horizontal; symbol Connector:Barrel_Jack -> Connector:Barrel_Jack_MountingPin
- J2: footprint (none) -> Connector_PinHeader_2.54mm:PinHeader_2x03_P2.54mm_Vertical
- J3: footprint (none) -> Connector_PinHeader_2.54mm:PinHeader_1x06_P2.54mm_Vertical_SMD_Pin1Left
- R1: footprint (none) -> Resistor_THT:R_Axial_DIN0207_L6.3mm_D2.5mm_P10.16mm_Horizontal
- RV1: footprint (none) -> Potentiometer_THT:Potentiometer_Alps_RK09K_Single_Vertical
- U1: footprint Package_DIP:DIP-28_W7.62mm -> Package_DIP:DIP-28_W7.62mm_Socket
- U10, U11, U12, U13, U14, U15, U16, U17, U18, U19, U4, U5, U6, U7, U8, U9: footprint (none) -> Package_DIP:DIP-16_W7.62mm
- U2: footprint (none) -> Package_DIP:DIP-8_W7.62mm_Socket
- U3: footprint (none) -> Package_TO_SOT_THT:TO-220-3_Horizontal_TabDown
- Y1: footprint (none) -> Crystal:Crystal_HC18-U_Vertical
Connections:
- net +5V: now also SW22.1 (A)
- net GND: now also J1.MP (MountPin), R3.2, R4.1, R5.1, SW21.2
- net RESET: now also SW21.1
- net SW_REG: now reaches U1.13 (PD7)
- net SW_REG: now also R3.1, SW22.2 (B)
- net at C2.1, J1.1: now also C3.1, U3.1 (IN)
- net at D105.1 (K): now also R4.2
- net at D121.1 (K): now also R5.2
- no-connect marks 2 -> 9
Other:
- note added: "Input / Output"
- moved on the sheet: C2, C3, C4, D105, D121, R1, RV1, U3

Commit message: Working on PCB layout.
Parts:
- J1: symbol Connector:Barrel_Jack_MountingPin -> Connector:Barrel_Jack_Switch
- J3: footprint Connector_PinHeader_2.54mm:PinHeader_1x06_P2.54mm_Vertical_SMD_Pin1Left -> Connector_PinHeader_2.54mm:PinHeader_1x06_P2.54mm_Vertical
Connections:
- net DISK_RCLK is gone; now on net DISP_RCLK: U1.26 (PC3)
- net +5V: no longer U4.10 (~SRCLR)
- net GND: now also J1.3; no longer J1.MP (MountPin)
- net RESET: now also U4.10 (~SRCLR)
- net VIN: now reaches C2.1, C3.1, J1.1, U3.1 (IN)
Other:
- moved on the sheet: J1
Changed lines of the file:
@@
 MISO
 $Comp
-L Connector:Barrel_Jack_MountingPin J1
+L Connector:Barrel_Jack_Switch J1
 U 1 1 5BD78797
 P 1200 1500
@@
 F 0 "J3" H 2670 8567 50  0000 C CNN
 F 1 "FDTI Serial" H 2670 8476 50  0000 C CNN
-F 2 "Connector_PinHeader_2.54mm:PinHeader_1x06_P2.54mm_Vertical_SMD_Pin1Left" H 2750 8150 50  0001 C CNN
+F 2 "Connector_PinHeader_2.54mm:PinHeader_1x06_P2.54mm_Vertical" H 2750 8150 50  0001 C CNN
 F 3 "~" H 2750 8150 50  0001 C CNN
 	1    2750 8150
@@
 	11000 6700 11500 6700
 $Comp
-L power:+5V #PWR011
-U 1 1 5C2CD5A8
-P 4800 2350
-F 0 "#PWR011" H 4800 2200 50  0001 C CNN
-F 1 "+5V" V 4815 2478 50  0000 L CNN
-F 2 "" H 4800 2350 50  0001 C CNN
-F 3 "" H 4800 2350 50  0001 C CNN
-	1    4800 2350
-	0    -1   -1   0
-$EndComp
-Wire Wire Line
-	4800 2350 4900 2350
-$Comp
 L 74xx:74HC595 U18
 U 1 1 5C5ADCB4
@@
 F8 "IO_INT" O R 6050 9850 50
 F9 "SDA" B R 6050 10000 50
-F10 "SCK" I R 6050 10150 50
+F10 "SCL" I R 6050 10150 50
 $EndSheet
 Wire Wire Line
@@
 DISP_CLK
 Text Label 3400 4300 2    50   ~ 0
-DISK_RCLK
+DISP_RCLK
 Wire Wire Line
 	2900 3100 3400 3100
@@
 SDA
 Text Label 6450 10150 2    50   ~ 0
-SCK
+SCL
 Text Label 3400 3200 2    50   ~ 0
 IO_INT
@@
 Connection ~ 2250 1250
 Wire Wire Line
-	1500 1750 1500 1850
+	1500 1600 1500 1500
+Connection ~ 1500 1600
 Wire Wire Line
-	1500 1850 1200 1850
-Wire Wire Line
-	1200 1850 1200 1800
-Connection ~ 1500 1750
+	4450 2350 4900 2350
+Text Label 4450 2350 0    50   ~ 0
+RESET
+Text Label 1850 1250 0    50   ~ 0
+VIN
 $EndSCHEMATC
