File: pcb/InputOutput.sch (KiCad schematic (older format))
At the start: 31 parts, among them J4 Power, J5 PortAB, SW1 A15, SW10 A10, SW11 A11, SW12 A9, SW13 A8, SW14 A7, SW15 A6, SW16 A5, SW17 A4, SW18 A3, SW19 A2, SW2 Run / Step, SW20 A1, SW3 A14, SW4 Reset / Clear, SW5 A13, SW6 Examine / Next, SW7 A12, SW8 Deposit / Next, SW9 A11, U20 74HC165, U21 74HC165, U22 74HC165, U23 MCP23017_SP

Commit message: Completed Schematic and assigned footprints.
Started PCB layout.
Parts:
- added C8: 10uF, LED_THT:LED_D5.0mm, symbol Device:CP
- C7: value 10uF -> 100nF; footprint (none) -> LED_THT:LED_D5.0mm
- J4: footprint (none) -> Connector_PinSocket_2.54mm:PinSocket_2x02_P2.54mm_Vertical
- J5: footprint (none) -> Connector_PinSocket_2.54mm:PinSocket_2x08_P2.54mm_Vertical
- R2: footprint (none) -> Resistor_THT:R_Axial_DIN0207_L6.3mm_D2.5mm_P10.16mm_Horizontal
- SW1, SW10, SW11, SW12, SW13, SW14, SW15, SW16, SW17, SW18, SW19, SW2, SW20, SW3, SW4, SW5, SW6, SW7, SW8, SW9: footprint (none) -> uvm:TOGGLE_SPDT_ON_ON_2MS
- U20, U21, U22: footprint (none) -> Package_DIP:DIP-16_W7.62mm
Connections:
- net +5V: now also SW1.2 (B), SW10.2 (B), SW11.2 (B), SW12.2 (B), SW13.2 (B), SW14.2 (B), SW15.2 (B), SW16.2 (B), SW17.2 (B), SW18.2 (B), SW19.2 (B), SW20.2 (B), SW3.2 (B), SW5.2 (B), SW7.2 (B), SW9.2 (B); no longer RN17.1 (common), RN19.1 (common)
- net GND: now also RN17.1 (common), RN19.1 (common)
- net at RN17.2 (R1): now also SW12.3 (C), U20.11 (A); no longer SW1.2 (B)
- net at SW1.3 (C), U20.6 (H): now also RN17.9 (R8)
- net at RN17.3 (R2): now also SW11.3 (C), U20.12 (B); no longer SW3.2 (B)
- net at SW3.3 (C), U20.5 (G): now also RN17.8 (R7)
- net at RN17.4 (R3): now also SW10.3 (C), U20.13 (C); no longer SW5.2 (B)
- net at SW5.3 (C), U20.4 (F): now also RN17.7 (R6)
- net at RN17.5 (R4): now also SW9.3 (C), U20.14 (D); no longer SW7.2 (B)
- net at SW7.3 (C), U20.3 (E): now also RN17.6 (R5)
- net at RN19.2 (R1): now also SW20.3 (C), U21.11 (A); no longer SW13.2 (B)
- net at SW13.3 (C), U21.6 (H): now also RN19.9 (R8)
- net at RN19.3 (R2): now also SW19.3 (C), U21.12 (B); no longer SW14.2 (B)
- net at SW14.3 (C), U21.5 (G): now also RN19.8 (R7)
- net at RN19.4 (R3): now also SW18.3 (C), U21.13 (C); no longer SW15.2 (B)
- net at SW15.3 (C), U21.4 (F): now also RN19.7 (R6)
- net at RN19.5 (R4): now also SW17.3 (C), U21.14 (D); no longer SW16.2 (B)
- net at SW16.3 (C), U21.3 (E): now also RN19.6 (R5)
- net at U23.21 (GPA0): now also J5.16 (Pin_16); no longer J5.9 (Pin_9)
- net at U23.22 (GPA1): now also J5.15 (Pin_15); no longer J5.10 (Pin_10)
- net at U23.23 (GPA2): now also J5.14 (Pin_14); no longer J5.11 (Pin_11)
- net at U23.24 (GPA3): now also J5.13 (Pin_13); no longer J5.12 (Pin_12)
- net at U23.25 (GPA4): now also J5.12 (Pin_12); no longer J5.13 (Pin_13)
- net at U23.26 (GPA5): now also J5.11 (Pin_11); no longer J5.14 (Pin_14)
- net at U23.27 (GPA6): now also J5.10 (Pin_10); no longer J5.15 (Pin_15)
- net at U23.28 (GPA7): now also J5.9 (Pin_9); no longer J5.16 (Pin_16)
- net at C7.2, J4.1 (Pin_1), J4.2 (Pin_2): now also C8.2
- net at C7.1, J4.3 (Pin_3), J4.4 (Pin_4): now also C8.1
- no-connect marks 4 -> 20
Other:
- moved on the sheet: C7, J5, RN17, RN19

Commit message: Working on PCB layout.
Parts:
- removed C8: 10uF, LED_THT:LED_D5.0mm, symbol Device:CP
- C7: footprint LED_THT:LED_D5.0mm -> Capacitor_THT:C_Disc_D6.0mm_W2.5mm_P5.00mm
- J5: symbol Connector_Generic:Conn_02x08_Top_Bottom -> Connector_Generic:Conn_02x08_Odd_Even
- SW1: value A15 -> A16
- SW10: value A10 -> A11
- SW11: value A11 -> A10
- SW3: value A14 -> A15
- SW5: value A13 -> A14
- SW7: value A12 -> A13
- SW9: value A11 -> A12
Connections:
- net +5V: now also C7.1, J4.3 (Pin_3), J4.4 (Pin_4)
- net GND: now also C7.2, J4.1 (Pin_1), J4.2 (Pin_2)
- net at U23.2 (GPB1): now also J5.3 (Pin_3); no longer J5.2 (Pin_2)
- net at U23.22 (GPA1): now also J5.14 (Pin_14); no longer J5.15 (Pin_15)
- net at U23.23 (GPA2): now also J5.12 (Pin_12); no longer J5.14 (Pin_14)
- net at U23.24 (GPA3): now also J5.10 (Pin_10); no longer J5.13 (Pin_13)
- net at U23.25 (GPA4): now also J5.8 (Pin_8); no longer J5.12 (Pin_12)
- net at U23.26 (GPA5): now also J5.6 (Pin_6); no longer J5.11 (Pin_11)
- net at U23.27 (GPA6): now also J5.4 (Pin_4); no longer J5.10 (Pin_10)
- net at U23.28 (GPA7): now also J5.2 (Pin_2); no longer J5.9 (Pin_9)
- net at U23.3 (GPB2): now also J5.5 (Pin_5); no longer J5.3 (Pin_3)
- net at U23.4 (GPB3): now also J5.7 (Pin_7); no longer J5.4 (Pin_4)
- net at U23.5 (GPB4): now also J5.9 (Pin_9); no longer J5.5 (Pin_5)
- net at U23.6 (GPB5): now also J5.11 (Pin_11); no longer J5.6 (Pin_6)
- net at U23.7 (GPB6): now also J5.13 (Pin_13); no longer J5.7 (Pin_7)
- net at U23.8 (GPB7): now also J5.15 (Pin_15); no longer J5.8 (Pin_8)
- net SCK renamed SCL
Other:
- moved on the sheet: C7, J4
Changed lines of the file:
@@
 AR Path="/5FA8FA07/5FB634CD" Ref="SW1"  Part="1"
 F 0 "SW1" H 3650 2435 50  0000 C CNN
-F 1 "A15" H 3650 2344 50  0000 C CNN
+F 1 "A16" H 3650 2344 50  0000 C CNN
 F 2 "uvm:TOGGLE_SPDT_ON_ON_2MS" H 3650 2150 50  0001 C CNN
 F 3 "" H 3650 2150 50  0001 C CNN
@@
 AR Path="/5FA8FA07/5FB634D4" Ref="SW3"  Part="1"
 F 0 "SW3" H 4250 2435 50  0000 C CNN
-F 1 "A14" H 4250 2344 50  0000 C CNN
+F 1 "A15" H 4250 2344 50  0000 C CNN
 F 2 "uvm:TOGGLE_SPDT_ON_ON_2MS" H 4250 2150 50  0001 C CNN
 F 3 "" H 4250 2150 50  0001 C CNN
@@
 AR Path="/5FA8FA07/5FB634DB" Ref="SW5"  Part="1"
 F 0 "SW5" H 4850 2435 50  0000 C CNN
-F 1 "A13" H 4850 2344 50  0000 C CNN
+F 1 "A14" H 4850 2344 50  0000 C CNN
 F 2 "uvm:TOGGLE_SPDT_ON_ON_2MS" H 4850 2150 50  0001 C CNN
 F 3 "" H 4850 2150 50  0001 C CNN
@@
 AR Path="/5FA8FA07/5FB634E2" Ref="SW7"  Part="1"
 F 0 "SW7" H 5450 2435 50  0000 C CNN
-F 1 "A12" H 5450 2344 50  0000 C CNN
+F 1 "A13" H 5450 2344 50  0000 C CNN
 F 2 "uvm:TOGGLE_SPDT_ON_ON_2MS" H 5450 2150 50  0001 C CNN
 F 3 "" H 5450 2150 50  0001 C CNN
@@
 AR Path="/5FA8FA07/5FB634E9" Ref="SW9"  Part="1"
 F 0 "SW9" H 6050 2435 50  0000 C CNN
-F 1 "A11" H 6050 2344 50  0000 C CNN
+F 1 "A12" H 6050 2344 50  0000 C CNN
 F 2 "uvm:TOGGLE_SPDT_ON_ON_2MS" H 6050 2150 50  0001 C CNN
 F 3 "" H 6050 2150 50  0001 C CNN
@@
 AR Path="/5FA8FA07/5FB634F0" Ref="SW10"  Part="1"
 F 0 "SW10" H 6650 2435 50  0000 C CNN
-F 1 "A10" H 6650 2344 50  0000 C CNN
+F 1 "A11" H 6650 2344 50  0000 C CNN
 F 2 "uvm:TOGGLE_SPDT_ON_ON_2MS" H 6650 2150 50  0001 C CNN
 F 3 "" H 6650 2150 50  0001 C CNN
@@
 AR Path="/5FA8FA07/5FB634F7" Ref="SW11"  Part="1"
 F 0 "SW11" H 7250 2435 50  0000 C CNN
-F 1 "A11" H 7250 2344 50  0000 C CNN
+F 1 "A10" H 7250 2344 50  0000 C CNN
 F 2 "uvm:TOGGLE_SPDT_ON_ON_2MS" H 7250 2150 50  0001 C CNN
 F 3 "" H 7250 2150 50  0001 C CNN
@@
 SDA
 Text HLabel 7950 6000 0    50   Input ~ 0
-SCK
+SCL
 $Comp
 L Connector_Generic:Conn_02x02_Top_Bottom J4
 U 1 1 61CB7B6F
-P 8300 4950
-F 0 "J4" V 8400 5100 50  0000 R CNN
-F 1 "Power" V 8300 5250 50  0000 R CNN
-F 2 "Connector_PinSocket_2.54mm:PinSocket_2x02_P2.54mm_Vertical" H 8300 4950 50  0001 C CNN
-F 3 "~" H 8300 4950 50  0001 C CNN
-	1    8300 4950
+P 9450 5150
+F 0 "J4" V 9550 5300 50  0000 R CNN
+F 1 "Power" V 9450 5450 50  0000 R CNN
+F 2 "Connector_PinSocket_2.54mm:PinSocket_2x02_P2.54mm_Vertical" H 9450 5150 50  0001 C CNN
+F 3 "~" H 9450 5150 50  0001 C CNN
+	1    9450 5150
 	0    -1   -1   0
 $EndComp
 Wire Wire Line
-	8300 4650 8300 4550
-Wire Wire Line
-	8300 5150 8300 5250
-Wire Wire Line
-	8300 5250 8400 5250
+	9450 4850 9450 4750
+Wire Wire Line
+	9450 5350 9450 5450
+Wire Wire Line
+	9450 5450 9550 5450
 $Comp
 L Device:C C7
 U 1 1 61D14A96
-P 9050 4900
-F 0 "C7" H 9165 4946 50  0000 L CNN
-F 1 "100nF" H 9165 4855 50  0000 L CNN
-F 2 "LED_THT:LED_D5.0mm" H 9088 4750 50  0001 C CNN
-F 3 "~" H 9050 4900 50  0001 C CNN
-	1    9050 4900
-	1    0    0    -1
-$EndComp
-Wire Wire Line
-	9050 4750 9050 4550
-Wire Wire Line
-	8300 4550 8400 4550
-Wire Wire Line
-	9050 5050 9050 5250
-Wire Wire Line
-	8400 5150 8400 5250
-Wire Wire Line
-	8400 4650 8400 4550
+P 9800 5100
+F 0 "C7" H 9915 5146 50  0000 L CNN
+F 1 "100nF" H 9915 5055 50  0000 L CNN
+F 2 "Capacitor_THT:C_Disc_D6.0mm_W2.5mm_P5.00mm" H 9838 4950 50  0001 C CNN
+F 3 "~" H 9800 5100 50  0001 C CNN
+	1    9800 5100
+	1    0    0    -1
+$EndComp
+Wire Wire Line
+	9800 4950 9800 4750
+Wire Wire Line
+	9450 4750 9550 4750
+Wire Wire Line
+	9800 5250 9800 5450
+Wire Wire Line
+	9550 5350 9550 5450
+Wire Wire Line
+	9550 4850 9550 4750
 $Comp
 L power:GND #PWR072
@@
 $EndComp
 $Comp
-L Connector_Generic:Conn_02x08_Top_Bottom J5
+L Connector_Generic:Conn_02x08_Odd_Even J5
 U 1 1 61DFF639
 P 10500 6650
@@
 NoConn ~ 4450 2050
 NoConn ~ 3850 2050
-Connection ~ 9050 4550
-Wire Wire Line
-	9050 4550 9200 4550
-Connection ~ 9050 5250
-Wire Wire Line
-	9050 5250 9200 5250
-Wire Wire Line
-	8400 4550 8600 4550
-Connection ~ 8400 4550
-Wire Wire Line
-	8400 5250 8600 5250
-Connection ~ 8400 5250
-$Comp
-L Device:CP C8
-U 1 1 5DD28219
-P 8600 4900
-F 0 "C8" H 8718 4946 50  0000 L CNN
-F 1 "10uF" H 8718 4855 50  0000 L CNN
-F 2 "LED_THT:LED_D5.0mm" H 8638 4750 50  0001 C CNN
-F 3 "~" H 8600 4900 50  0001 C CNN
-	1    8600 4900
-	1    0    0    -1
-$EndComp
-Wire Wire Line
-	8600 5050 8600 5250
-Connection ~ 8600 5250
-Wire Wire Line
-	8600 5250 9050 5250
-Wire Wire Line
-	8600 4750 8600 4550
-Connection ~ 8600 4550
-Wire Wire Line
-	8600 4550 9050 4550
+$Comp
+L power:+5V #PWR0101
+U 1 1 5C0B7F75
+P 10250 4650
+F 0 "#PWR0101" H 10250 4500 50  0001 C CNN
+F 1 "+5V" H 10265 4823 50  0000 C CNN
+F 2 "" H 10250 4650 50  0001 C CNN
+F 3 "" H 10250 4650 50  0001 C CNN
+	1    10250 4650
+	1    0    0    -1
+$EndComp
+$Comp
+L power:GND #PWR0102
+U 1 1 5C0B7FEC
+P 10250 5600
+F 0 "#PWR0102" H 10250 5350 50  0001 C CNN
+F 1 "GND" H 10255 5427 50  0000 C CNN
+F 2 "" H 10250 5600 50  0001 C CNN
+F 3 "" H 10250 5600 50  0001 C CNN
+	1    10250 5600
+	1    0    0    -1
+$EndComp
+Wire Wire Line
+	10250 5450 10250 5600
+Wire Wire Line
+	10250 4750 10250 4650
+Text Label 9900 4750 0    50   ~ 0
+VPORT
+Wire Wire Line
+	9800 4750 10250 4750
+Wire Wire Line
+	9800 5450 10250 5450
+Wire Wire Line
+	9550 5450 9800 5450
+Connection ~ 9550 5450
+Connection ~ 9800 5450
+Wire Wire Line
+	9800 4750 9550 4750
+Connection ~ 9800 4750
+Connection ~ 9550 4750
 $EndSCHEMATC

Commit message: Completed PCB Layout.
Parts:
- SW1: value A16 -> A15
- SW10: value A11 -> A10
- SW11: value A10 -> A9
- SW12: value A9 -> A8
- SW13: value A8 -> A7
- SW14: value A7 -> A6
- SW15: value A6 -> A5
- SW16: value A5 -> A4
- SW17: value A4 -> A3
- SW18: value A3 -> A2
- SW19: value A2 -> A1
- SW20: value A1 -> A0
- SW3: value A15 -> A14
- SW5: value A14 -> A13
- SW7: value A13 -> A12
- SW9: value A12 -> A11
Changed lines of the file:
@@
 AR Path="/5FA8FA07/5FB634CD" Ref="SW1"  Part="1"
 F 0 "SW1" H 3650 2435 50  0000 C CNN
-F 1 "A16" H 3650 2344 50  0000 C CNN
+F 1 "A15" H 3650 2344 50  0000 C CNN
 F 2 "uvm:TOGGLE_SPDT_ON_ON_2MS" H 3650 2150 50  0001 C CNN
 F 3 "" H 3650 2150 50  0001 C CNN
@@
 AR Path="/5FA8FA07/5FB634D4" Ref="SW3"  Part="1"
 F 0 "SW3" H 4250 2435 50  0000 C CNN
-F 1 "A15" H 4250 2344 50  0000 C CNN
+F 1 "A14" H 4250 2344 50  0000 C CNN
 F 2 "uvm:TOGGLE_SPDT_ON_ON_2MS" H 4250 2150 50  0001 C CNN
 F 3 "" H 4250 2150 50  0001 C CNN
@@
 AR Path="/5FA8FA07/5FB634DB" Ref="SW5"  Part="1"
 F 0 "SW5" H 4850 2435 50  0000 C CNN
-F 1 "A14" H 4850 2344 50  0000 C CNN
+F 1 "A13" H 4850 2344 50  0000 C CNN
 F 2 "uvm:TOGGLE_SPDT_ON_ON_2MS" H 4850 2150 50  0001 C CNN
 F 3 "" H 4850 2150 50  0001 C CNN
@@
 AR Path="/5FA8FA07/5FB634E2" Ref="SW7"  Part="1"
 F 0 "SW7" H 5450 2435 50  0000 C CNN
-F 1 "A13" H 5450 2344 50  0000 C CNN
+F 1 "A12" H 5450 2344 50  0000 C CNN
 F 2 "uvm:TOGGLE_SPDT_ON_ON_2MS" H 5450 2150 50  0001 C CNN
 F 3 "" H 5450 2150 50  0001 C CNN
@@
 AR Path="/5FA8FA07/5FB634E9" Ref="SW9"  Part="1"
 F 0 "SW9" H 6050 2435 50  0000 C CNN
-F 1 "A12" H 6050 2344 50  0000 C CNN
+F 1 "A11" H 6050 2344 50  0000 C CNN
 F 2 "uvm:TOGGLE_SPDT_ON_ON_2MS" H 6050 2150 50  0001 C CNN
 F 3 "" H 6050 2150 50  0001 C CNN
@@
 AR Path="/5FA8FA07/5FB634F0" Ref="SW10"  Part="1"
 F 0 "SW10" H 6650 2435 50  0000 C CNN
-F 1 "A11" H 6650 2344 50  0000 C CNN
+F 1 "A10" H 6650 2344 50  0000 C CNN
 F 2 "uvm:TOGGLE_SPDT_ON_ON_2MS" H 6650 2150 50  0001 C CNN
 F 3 "" H 6650 2150 50  0001 C CNN
@@
 AR Path="/5FA8FA07/5FB634F7" Ref="SW11"  Part="1"
 F 0 "SW11" H 7250 2435 50  0000 C CNN
-F 1 "A10" H 7250 2344 50  0000 C CNN
+F 1 "A9" H 7250 2344 50  0000 C CNN
 F 2 "uvm:TOGGLE_SPDT_ON_ON_2MS" H 7250 2150 50  0001 C CNN
 F 3 "" H 7250 2150 50  0001 C CNN
@@
 AR Path="/5FA8FA07/5FB634FE" Ref="SW12"  Part="1"
 F 0 "SW12" H 7850 2435 50  0000 C CNN
-F 1 "A9" H 7850 2344 50  0000 C CNN
+F 1 "A8" H 7850 2344 50  0000 C CNN
 F 2 "uvm:TOGGLE_SPDT_ON_ON_2MS" H 7850 2150 50  0001 C CNN
 F 3 "" H 7850 2150 50  0001 C CNN
@@
 AR Path="/5FA8FA07/5FB63577" Ref="SW13"  Part="1"
 F 0 "SW13" H 9500 2435 50  0000 C CNN
-F 1 "A8" H 9500 2344 50  0000 C CNN
+F 1 "A7" H 9500 2344 50  0000 C CNN
 F 2 "uvm:TOGGLE_SPDT_ON_ON_2MS" H 9500 2150 50  0001 C CNN
 F 3 "" H 9500 2150 50  0001 C CNN
@@
 AR Path="/5FA8FA07/5FB6357E" Ref="SW14"  Part="1"
 F 0 "SW14" H 10100 2435 50  0000 C CNN
-F 1 "A7" H 10100 2344 50  0000 C CNN
+F 1 "A6" H 10100 2344 50  0000 C CNN
 F 2 "uvm:TOGGLE_SPDT_ON_ON_2MS" H 10100 2150 50  0001 C CNN
 F 3 "" H 10100 2150 50  0001 C CNN
@@
 AR Path="/5FA8FA07/5FB63585" Ref="SW15"  Part="1"
 F 0 "SW15" H 10700 2435 50  0000 C CNN
-F 1 "A6" H 10700 2344 50  0000 C CNN
+F 1 "A5" H 10700 2344 50  0000 C CNN
 F 2 "uvm:TOGGLE_SPDT_ON_ON_2MS" H 10700 2150 50  0001 C CNN
 F 3 "" H 10700 2150 50  0001 C CNN
@@
 AR Path="/5FA8FA07/5FB6358C" Ref="SW16"  Part="1"
 F 0 "SW16" H 11300 2435 50  0000 C CNN
-F 1 "A5" H 11300 2344 50  0000 C CNN
+F 1 "A4" H 11300 2344 50  0000 C CNN
 F 2 "uvm:TOGGLE_SPDT_ON_ON_2MS" H 11300 2150 50  0001 C CNN
 F 3 "" H 11300 2150 50  0001 C CNN
@@
 AR Path="/5FA8FA07/5FB63593" Ref="SW17"  Part="1"
 F 0 "SW17" H 11900 2435 50  0000 C CNN
-F 1 "A4" H 11900 2344 50  0000 C CNN
+F 1 "A3" H 11900 2344 50  0000 C CNN
 F 2 "uvm:TOGGLE_SPDT_ON_ON_2MS" H 11900 2150 50  0001 C CNN
 F 3 "" H 11900 2150 50  0001 C CNN
@@
 AR Path="/5FA8FA07/5FB6359A" Ref="SW18"  Part="1"
 F 0 "SW18" H 12500 2435 50  0000 C CNN
-F 1 "A3" H 12500 2344 50  0000 C CNN
+F 1 "A2" H 12500 2344 50  0000 C CNN
 F 2 "uvm:TOGGLE_SPDT_ON_ON_2MS" H 12500 2150 50  0001 C CNN
 F 3 "" H 12500 2150 50  0001 C CNN
@@
 AR Path="/5FA8FA07/5FB635A1" Ref="SW19"  Part="1"
 F 0 "SW19" H 13100 2435 50  0000 C CNN
-F 1 "A2" H 13100 2344 50  0000 C CNN
+F 1 "A1" H 13100 2344 50  0000 C CNN
 F 2 "uvm:TOGGLE_SPDT_ON_ON_2MS" H 13100 2150 50  0001 C CNN
 F 3 "" H 13100 2150 50  0001 C CNN
@@
 AR Path="/5FA8FA07/5FB635A8" Ref="SW20"  Part="1"
 F 0 "SW20" H 13700 2435 50  0000 C CNN
-F 1 "A1" H 13700 2344 50  0000 C CNN
+F 1 "A0" H 13700 2344 50  0000 C CNN
 F 2 "uvm:TOGGLE_SPDT_ON_ON_2MS" H 13700 2150 50  0001 C CNN
 F 3 "" H 13700 2150 50  0001 C CNN
