File: pcb/uvm.kicad_pcb (KiCad board)
At the start: 2 copper layers, 206 parts, among them J1 Barrel_Jack, J2 ICSP, J3 FDTI Serial, J4 Power, J5 PortAB, SW1 A15, SW10 A10, SW11 A11, SW12 A9, SW13 A8, SW14 A7, SW15 A6, SW16 A5, SW17 A4, SW18 A3, SW19 A2, SW2 Run / Step, SW20 A1, SW21 RESET, SW22 REG Select, SW3 A14, SW4 Reset / Clear, SW5 A13, SW6 Examine / Next, SW7 A12, SW8 Deposit / Next, SW9 A11, U1 ATmega328P-PU, U10 74HC595, U11 74HC595, U12 74HC595, U13 74HC595, U14 74HC595, U15 74HC595, U16 74HC595, U17 74HC595, U18 74HC595, U19 74HC595, U2 23LCV512, U20 74HC165, U21 74HC165, U22 74HC165, U23 MCP23017_SP, U3 L7805, U4 74HC595, U5 74HC595, U6 74HC595, U7 74HC595, U8 74HC595, U9 74HC595, Y1 16MHz

Commit message: Working on PCB layout.
Parts:
- removed C8: 10uF, LED_THT:LED_D5.0mm
- C7: footprint LED_THT:LED_D5.0mm -> Capacitor_THT:C_Disc_D6.0mm_W2.5mm_P5.00mm
- SW1: value A15 -> A16
- SW10: value A10 -> A11
- SW11: value A11 -> A10
- SW3: value A14 -> A15
- SW5: value A13 -> A14
- SW7: value A12 -> A13
- SW9: value A11 -> A12
- moved D33 215.6 mm to (53.6, 82.5)
- moved D5 215.4 mm to (53.6, 48.3)
- moved D29 206.1 mm to (59.9, 71.1)
- moved D37 198.8 mm to (53.6, 94.0)
- moved D22 191.6 mm to (72.6, 48.3)
- moved D17 191.2 mm to (59.9, 36.8)
- moved D49 189.8 mm to (59.9, 82.5)
- moved D18 189.5 mm to (72.6, 36.8)
- moved U5 187.3 mm to (32.0, 50.8), turned to 90 degrees
- moved D50 184.2 mm to (72.6, 82.5)
- moved D53 180.8 mm to (59.9, 94.0)
- moved D41 180.5 mm to (53.6, 105.4)
- moved D51 178.5 mm to (85.3, 82.5)
- moved U4 178.2 mm to (32.0, 39.4), turned to 90 degrees
- moved D42 176.3 mm to (66.3, 105.4)
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Connections:
- net Net-(C2-Pad1) renamed /VIN
- C7 pad 1: Net-(C7-Pad1) -> +5V
- C7 pad 2: Net-(C7-Pad2) -> GND
- J1 pad 3: (no net) -> GND
- J4 pad 1: Net-(C7-Pad2) -> GND
- J4 pad 2: Net-(C7-Pad2) -> GND
- J4 pad 3: Net-(C7-Pad1) -> +5V
- J4 pad 4: Net-(C7-Pad1) -> +5V
- U1 pad 26: /DISK_RCLK -> /DISP_RCLK
- U23 pad 12: /SCK -> /SCL
- U23 pad 2: Net-(J5-Pad2) -> Net-(J5-Pad3)
- U23 pad 22: Net-(J5-Pad15) -> Net-(J5-Pad14)
- U23 pad 23: Net-(J5-Pad14) -> Net-(J5-Pad12)
- U23 pad 24: Net-(J5-Pad13) -> Net-(J5-Pad10)
- U23 pad 25: Net-(J5-Pad12) -> Net-(J5-Pad8)
- U23 pad 26: Net-(J5-Pad11) -> Net-(J5-Pad6)
- U23 pad 27: Net-(J5-Pad10) -> Net-(J5-Pad4)
- U23 pad 28: Net-(J5-Pad9) -> Net-(J5-Pad2)
- U23 pad 3: Net-(J5-Pad3) -> Net-(J5-Pad5)
- U23 pad 4: Net-(J5-Pad4) -> Net-(J5-Pad7)
- U23 pad 5: Net-(J5-Pad5) -> Net-(J5-Pad9)
- U23 pad 6: Net-(J5-Pad6) -> Net-(J5-Pad11)
- U23 pad 7: Net-(J5-Pad7) -> Net-(J5-Pad13)
- U23 pad 8: Net-(J5-Pad8) -> Net-(J5-Pad15)
- U4 pad 10: +5V -> /RESET
Routing:
- net /RESET: track 0.00 -> 647.9 mm, vias 0 -> 2
- net /DISP_RCLK: track 0.00 -> 559.8 mm
- net /DISP_CLK: track 0.00 -> 554.3 mm
- net /DISP_EN: track 0.00 -> 529.4 mm, vias 0 -> 1
- net /D_REG_IN: track 0.00 -> 269.0 mm, vias 0 -> 1
- net /SW_REG: track 0.00 -> 226.0 mm, vias 0 -> 1
- net /D_PC_IN: track 0.00 -> 205.9 mm
- net /IO_INT: track 0.00 -> 164.1 mm
- net Net-(U12-Pad9): track 0.00 -> 146.0 mm, vias 0 -> 1
- net Net-(U18-Pad9): track 0.00 -> 144.6 mm
- net /D_STATUS_IN: track 0.00 -> 144.0 mm
- net Net-(U14-Pad9): track 0.00 -> 141.6 mm
- net Net-(RN18-Pad9): track 0.00 -> 138.1 mm
- net /D_DATA_IN: track 0.00 -> 133.5 mm
- net /D_ADDR_IN: track 0.00 -> 123.9 mm, vias 0 -> 1
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Other:
- board outline added: 246.4 x 127 mm
- net class Vin added: clearance 0.4, trace_width 0.6, via_dia 0.8, via_drill 0.4

Commit message: Completed PCB Layout.
Parts:
- SW1: value A16 -> A15
- SW10: value A11 -> A10
- SW11: value A10 -> A9
- SW12: value A9 -> A8
- SW13: value A8 -> A7
- SW14: value A7 -> A6
- SW15: value A6 -> A5
- SW16: value A5 -> A4
- SW17: value A4 -> A3
- SW18: value A3 -> A2
- SW19: value A2 -> A1
- SW20: value A1 -> A0
- SW3: value A15 -> A14
- SW5: value A14 -> A13
- SW7: value A13 -> A12
- SW9: value A12 -> A11
- moved R3 17.5 mm to (114.9, 41.9), turned to 90 degrees
- moved R5 13.9 mm to (207.5, 72.4), turned to 90 degrees
- moved SW21 13.0 mm to (223.6, 125.5)
- moved R1 12.5 mm to (233.7, 135.1), turned to 90 degrees
- moved R4 5.73 mm to (204.2, 72.4), turned to 90 degrees
- moved SW6 4.80 mm to (164.6, 107.8)
- moved SW8 4.23 mm to (154.9, 107.7)
- moved R2 1.78 mm to (116.8, 124.5)
- moved D105 1.52 mm to (198.1, 67.3)
- moved D121 1.02 mm to (210.8, 67.3)
- moved SW22 0.89 mm to (106.0, 31.8)
Routing:
- net GND: track 0.00 -> 221.7 mm, vias 0 -> 7
- net /SW_REG: track 226.0 -> 177.0 mm
- net +5V: track 0.00 -> 38.2 mm, vias 0 -> 6
- net /RESET: track 647.9 -> 668.4 mm
- net /RX: track 0.00 -> 12.6 mm
- net Net-(RN18-Pad7): track 120.7 -> 112.6 mm
- net Net-(RN18-Pad6): track 107.9 -> 101.7 mm
- net Net-(RN18-Pad9): track 138.1 -> 134.5 mm
- net /D_DATA_IN: track 133.5 -> 130.1 mm
- net Net-(D105-Pad2): track 80.1 -> 83.2 mm
- net Net-(U4-Pad9): track 23.9 -> 21.6 mm
- net Net-(RN18-Pad8): track 123.5 -> 121.2 mm
- net Net-(D105-Pad1): track 6.35 -> 8.27 mm
- net Net-(D121-Pad1): track 6.35 -> 7.64 mm
- net Net-(D121-Pad2): track 61.1 -> 60.0 mm
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- added copper zone on F.Cu, net +5V
- added copper zone on B.Cu, net GND
Other:
- board size 246.4 x 127 mm -> 245 x 126 mm
- board text added: "+5V"
- board text added: "0"
- board text added: "1"
- board text added: "128"
- board text added: "16"
- board text added: "2"
- board text added: "3"
- board text added: "32"
- board text added: "4"
- board text added: "5"
- board text added: "6"
- board text added: "64"
- board text added: "7"
- board text added: "7V-12V"
- board text added: "8"
- board text added: "9"
- board text added: "A"
- board text added: "A0"
- board text added: "A1"
- board text added: "A10"
- board text added: "A11"
- board text added: "A12"
- board text added: "A13"
- board text added: "A14"
- board text added: "A15"
- board text added: "A2"
- board text added: "A3"
- board text added: "A4"
- board text added: "A5"
- board text added: "A6"
- board text added: "A7"
- board text added: "A8"
- board text added: "A9"
- board text added: "Address"
- board text added: "B"
- board text added: "C"
- board text added: "CLEAR"
- board text added: "D"
- board text added: "Data @ Address"
- board text added: "Deposit"
- board text added: "Deposit Next"
- board text added: "E"
- board text added: "Examine"
- board text added: "Examine Next"
- board text added: "Extended Registers AX = 4&5 BX = 6&7 CX = 8&9 DX = A&B EX = C&D FX = E&F"
- board text added: "F"
- board text added: "GND"
- board text added: "HALT"
- board text added: "IO Ports"
- board text added: "Instruction @ PC"
- board text added: "Program Counter"
- board text added: "RESET"
- board text added: "RUN"
- board text added: "RUN SPEED"
- board text added: "Registers"
- board text added: "STEP"
- board text added: "uVM 8-Bit Computer https://github.com/sam159/uVM Sam Stevens 2018"
